File: Extension.sch (KiCad schematic (older format))
At the start: 2 parts, among them J7 CLT-110-02-F-D-BE-A, J8 CLT-106-02-F-D-BE-A

Commit message: PVT
Connections:
- net ~UART_CTS renamed KICKER_N
- net ~UART_RTS renamed KICKER_P
Changed lines of the file:
@@
 encoding utf-8
 Sheet 6 24
-Title "Phoenix DVT"
-Date "2020-05-18"
+Title "Phoenix PVT"
+Date "2020-07-19"
 Rev "1"
 Comp ""
@@
 $EndDescr
 $Comp
-L supply-alias:GND #PWR0168
+L supply-alias:GND #PWR0155
 U 1 1 5E837C95
 P 4900 4100
-F 0 "#PWR0168" H 4900 3850 50  0001 C CNN
+F 0 "#PWR0155" H 4900 3850 50  0001 C CNN
 F 1 "GND" H 4900 3950 50  0000 C CNN
 F 2 "" H 4900 4100 50  0001 C CNN
@@
 Text HLabel 6600 3500 2    50   Output ~ 0
 UART_RX
-Text HLabel 4500 3500 0    50   Input ~ 0
-~UART_RTS
-Text HLabel 6600 3600 2    50   Output ~ 0
-~UART_CTS
-Wire Wire Line
-	4500 3500 5300 3500
-Wire Wire Line
-	5800 3600 6600 3600
 $Comp
 L Connector_Generic:Conn_02x10_Odd_Even J7
@@
 $EndComp
 $Comp
-L supply-alias:GND #PWR0174
+L supply-alias:GND #PWR0161
 U 1 1 5EDE3469
 P 6200 4100
-F 0 "#PWR0174" H 6200 3850 50  0001 C CNN
+F 0 "#PWR0161" H 6200 3850 50  0001 C CNN
 F 1 "GND" H 6200 3950 50  0000 C CNN
 F 2 "" H 6200 4100 50  0001 C CNN
@@
 $EndComp
 $Comp
-L supply-alias:GND #PWR0169
+L supply-alias:GND #PWR0156
 U 1 1 5EDB997F
 P 4900 5600
-F 0 "#PWR0169" H 4900 5350 50  0001 C CNN
+F 0 "#PWR0156" H 4900 5350 50  0001 C CNN
 F 1 "GND" H 4900 5450 50  0000 C CNN
 F 2 "" H 4900 5600 50  0001 C CNN
@@
 $EndComp
 $Comp
-L supply-alias:GND #PWR0175
+L supply-alias:GND #PWR0162
 U 1 1 5EDC1BF5
 P 6200 5600
-F 0 "#PWR0175" H 6200 5350 50  0001 C CNN
+F 0 "#PWR0162" H 6200 5350 50  0001 C CNN
 F 1 "GND" H 6200 5450 50  0000 C CNN
 F 2 "" H 6200 5600 50  0001 C CNN
@@
 	4900 3000 4900 4100
 $Comp
-L supply-value:+1V8 #PWR0172
+L supply-value:+1V8 #PWR0159
 U 1 1 5EE31384
 P 6000 4900
-F 0 "#PWR0172" H 6000 4750 50  0001 C CNN
+F 0 "#PWR0159" H 6000 4750 50  0001 C CNN
 F 1 "+1V8" H 6000 5040 50  0000 C CNN
 F 2 "" H 6000 4900 50  0001 C CNN
@@
 	5300 5500 4500 5500
 $Comp
-L supply-value:+5V #PWR0170
+L supply-value:+5V #PWR0157
 U 1 1 5F286AC8
 P 5100 2900
-F 0 "#PWR0170" H 5100 2750 50  0001 C CNN
+F 0 "#PWR0157" H 5100 2750 50  0001 C CNN
 F 1 "+5V" H 5100 3040 50  0000 C CNN
 F 2 "" H 5100 2900 50  0001 C CNN
@@
 	5800 3000 6000 3000
 $Comp
-L supply-value:+3V3 #PWR0171
+L supply-value:+3V3 #PWR0158
 U 1 1 5F28A290
 P 6000 2900
-F 0 "#PWR0171" H 6000 2750 50  0001 C CNN
+F 0 "#PWR0158" H 6000 2750 50  0001 C CNN
 F 1 "+3V3" H 6000 3040 50  0000 C CNN
 F 2 "" H 6000 2900 50  0001 C CNN
@@
 $EndComp
 $Comp
-L supply-alias:VBAT #PWR0173
+L supply-alias:VBAT #PWR0160
 U 1 1 5F337487
 P 6200 2900
-F 0 "#PWR0173" H 6200 2750 50  0001 C CNN
+F 0 "#PWR0160" H 6200 2750 50  0001 C CNN
 F 1 "VBAT" H 6200 3040 50  0000 C CNN
 F 2 "" H 6200 2900 50  0001 C CNN
@@
 Wire Wire Line
 	5300 3700 4500 3700
+Text HLabel 4500 3500 0    50   BiDi ~ 0
+KICKER_P
+Text HLabel 6600 3600 2    50   BiDi ~ 0
+KICKER_N
+Wire Wire Line
+	6600 3600 5800 3600
+Wire Wire Line
+	5300 3500 4500 3500
 $EndSCHEMATC
