File: PowerSequencer.sch (KiCad schematic (older format))
At the start: 23 parts, among them J1 B4B-ZR, Q1 BSS138W, Q2 BSS138W, Q3 BSS138W, U1 SLG46826G, U2 TLA2024IRUGR

Commit message: PVT
Parts:
- removed U2: TLA2024IRUGR, IC-QFN:QFN10_1.5x2.0_P0.5_001, symbol analog-ti:TLA2024
- added C6: 1u, Capacitor-Chip:C_CHIP_1005_Hand_NoSilk, symbol passive:C
- added U2: ADS1015IDGSR, IC-SOP:VSSOP10_3.0x3.0_P0.5, symbol analog-ti:ADS1015
- U1: footprint IC-SOP:TSSOP20-W4.4_Hand -> IC-SOP:TSSOP20-W4.4; Supplier Mouser -> (none)
Connections:
- net +3V3A: now also U2.8 (VDD); no longer Q3.1 (G)
- net ESW_IS: no longer U1.2 (IO13/ACMP1H_IN)
- net GND: now also C6.2, U2.1 (ADDR), U2.3 (GND)
- net TEMP_MON: now also U2.7 (AIN3)
- net VSTBY: now also Q3.1 (G)
- net at Q2.2 (S): now also U2.5 (AIN1)
- net at Q1.2 (S): now also U2.4 (AIN0)
- net ESW_IS_CLAMPED: now reaches Q3.2 (S)
- net ESW_IS_CLAMPED: now also U1.2 (IO13/ACMP1H_IN), C6.1, U2.6 (AIN2)
- net ~GP_FAULT renamed ~FPGA_STOP
- net ~SW_UNDECIDED renamed ~SW_WAKE_SLEEP
- new net ADC3_SCL: U2.10 (SCL)
- new net ADC3_SDA: U2.9 (SDA)
Other:
- note added: "ADC3 (controller by Processor)"
- note added: "I2C Address : 0b0001000"
- note removed: "ADC (controller by Processor)"
Changed lines of the file:
@@
 encoding utf-8
 Sheet 2 24
-Title "Phoenix DVT"
-Date "2020-05-18"
+Title "Phoenix PVT"
+Date "2020-07-19"
 Rev "1"
 Comp ""
@@
 F 0 "U1" H 3500 3250 50  0000 C CNN
 F 1 "SLG46826G" H 3500 1350 50  0000 C CNN
-F 2 "IC-SOP:TSSOP20-W4.4_Hand" H 3500 2300 50  0001 C CNN
+F 2 "IC-SOP:TSSOP20-W4.4" H 3500 2300 50  0001 C CNN
 F 3 "" H 3500 2300 50  0001 C CNN
 F 4 "SLG46826G" H 3500 2300 50  0001 C CNN "PartName"
-F 5 "Mouser" H 3500 2300 50  0001 C CNN "Supplier"
+F 5 "" H 3500 2300 50  0001 C CNN "Supplier"
 	1    3500 2300
 	1    0    0    -1
@@
 Wire Wire Line
 	2000 2100 2900 2100
-Text HLabel 5000 3000 2    50   Input ~ 0
+Text HLabel 10200 2900 2    50   Input ~ 0
 ESW_IS
 Wire Wire Line
-	5000 3000 4100 3000
+	4300 3000 4100 3000
 Text HLabel 5000 2500 2    50   Input ~ 0
 ~SW_POWER
-Wire Wire Line
-	5000 2000 4100 2000
 $Comp
 L supply-alias:VSYS #PWR013
@@
 Wire Wire Line
 	4100 2400 5000 2400
-Text HLabel 5000 2000 2    50   Input ~ 0
-~SW_UNDECIDED
 Wire Wire Line
 	4100 2500 5000 2500
@@
 	4300 2700 4100 2700
 Text HLabel 5000 1500 2    50   Output ~ 0
-~GP_FAULT
+~FPGA_STOP
 Wire Wire Line
 	5000 1500 4600 1500
@@
 $EndComp
 Text HLabel 8700 1500 2    50   BiDi ~ 0
-ADC_SCL
+ADC3_SCL
 Text HLabel 8700 1700 2    50   BiDi ~ 0
-ADC_SDA
+ADC3_SDA
 $Comp
 L supply-value:+3V3A #PWR?
@@
 Connection ~ 9200 2000
 Wire Wire Line
-	9200 2000 9700 2000
-Wire Wire Line
-	9700 2000 9700 2700
-Wire Wire Line
-	9500 2900 8100 2900
+	9500 2900 9300 2900
 Wire Wire Line
 	8100 2900 8100 2300
@@
 Wire Wire Line
 	8000 2500 8000 3200
-Wire Wire Line
-	9900 2900 10200 2900
 Wire Wire Line
 	8000 3200 10200 3200
@@
 	6000 4000 6000 500
 Text Notes 6100 800  0    100  ~ 20
-ADC (controller by Processor)
+ADC3 (controller by Processor)
 Text Label 10200 2300 0    50   ~ 0
 VBAT_IN_MON
 Text Label 10200 3200 0    50   ~ 0
 TEMP_MON
-Text Label 4300 3000 0    50   ~ 0
-ESW_IS
-Text Label 10200 2900 0    50   ~ 0
-ESW_IS
 $Comp
 L transistor-mos:Q_NMOS_GSD Q?
@@
 Wire Wire Line
 	8300 2300 8500 2300
-$Comp
-L analog-ti:TLA2024 U?
-U 1 1 5F102B71
+Wire Wire Line
+	7900 1700 8700 1700
+Wire Wire Line
+	7900 1500 8700 1500
+$Comp
+L analog-ti:ADS1015 U2
+U 1 1 5F6F676D
 P 7500 2000
-AR Path="/5E83D44B/5F102B71" Ref="U?"  Part="1"
-AR Path="/5EBDE4A1/5F102B71" Ref="U?"  Part="1"
-AR Path="/5E8151C7/5F102B71" Ref="U2"  Part="1"
-AR Path="/5E9E174E/5F102B71" Ref="U?"  Part="1"
 F 0 "U2" H 7500 2650 50  0000 C CNN
-F 1 "TLA2024IRUGR" H 7500 1350 50  0000 C CNN
-F 2 "IC-QFN:QFN10_1.5x2.0_P0.5_001" H 7500 2000 50  0001 C CNN
+F 1 "ADS1015IDGSR" H 7500 1350 50  0000 C CNN
+F 2 "IC-SOP:VSSOP10_3.0x3.0_P0.5" H 7500 2000 50  0001 C CNN
 F 3 "" H 7500 2000 50  0001 C CNN
-F 4 "TLA2024IRUGR" H 7500 2000 50  0001 C CNN "PartName"
+F 4 "ADS1015IDGSR" H 7500 2000 50  0001 C CNN "PartName"
 	1    7500 2000
 	1    0    0    -1
 $EndComp
 Wire Wire Line
-	7900 1700 8700 1700
-Wire Wire Line
-	7900 1500 8700 1500
+	10200 2900 9900 2900
+Wire Wire Line
+	9700 2700 9700 2000
+$Comp
+L supply-alias:VSTBY #PWR018
+U 1 1 5EF3AEA3
+P 9700 2000
+F 0 "#PWR018" H 9700 1850 50  0001 C CNN
+F 1 "VSTBY" H 9700 2140 50  0000 C CNN
+F 2 "" H 9700 2000 50  0001 C CNN
+F 3 "" H 9700 2000 50  0001 C CNN
+	1    9700 2000
+	1    0    0    -1
+$EndComp
+Text Label 9200 2900 2    50   ~ 0
+ESW_IS_CLAMPED
+Text Label 4300 3000 0    50   ~ 0
+ESW_IS_CLAMPED
+$Comp
+L supply-alias:GND #PWR?
+U 1 1 5EF74F50
+P 9300 3600
+AR Path="/5E314B49/5EF74F50" Ref="#PWR?"  Part="1"
+AR Path="/5F5738E6/5EF74F50" Ref="#PWR?"  Part="1"
+AR Path="/5E8151C7/5EF74F50" Ref="#PWR017"  Part="1"
+F 0 "#PWR017" H 9300 3350 50  0001 C CNN
+F 1 "GND" H 9300 3450 50  0000 C CNN
+F 2 "" H 9300 3600 50  0001 C CNN
+F 3 "" H 9300 3600 50  0001 C CNN
+	1    9300 3600
+	1    0    0    -1
+$EndComp
+Wire Wire Line
+	9300 3600 9300 3500
+$Comp
+L passive:C C?
+U 1 1 5EF74F58
+P 9300 3400
+AR Path="/5E83D44B/5EF74F58" Ref="C?"  Part="1"
+AR Path="/5E8151C7/5EF74F58" Ref="C6"  Part="1"
+AR Path="/5E314B49/5EF74F58" Ref="C?"  Part="1"
+F 0 "C6" H 9400 3450 50  0000 L CNN
+F 1 "1u" H 9400 3350 50  0000 L CNN
+F 2 "Capacitor-Chip:C_CHIP_1005_Hand_NoSilk" H 9400 3300 50  0001 C CNN
+F 3 "" H 9325 3500 50  0001 C CNN
+F 4 "TMK105BJ105MV-F" H 9300 3400 50  0001 C CNN "PartName"
+	1    9300 3400
+	1    0    0    -1
+$EndComp
+Wire Wire Line
+	9300 2900 9300 3300
+Connection ~ 9300 2900
+Wire Wire Line
+	9300 2900 8100 2900
+Text HLabel 5000 2000 2    50   Input ~ 0
+~SW_WAKE_SLEEP
+Wire Wire Line
+	5000 2000 4100 2000
+Text Notes 3000 3500 0    50   ~ 0
+I2C Address : 0b0001000
 $EndSCHEMATC
