File: Power2.sch (KiCad schematic (older format))
At the start: 61 parts, among them U10 LM26480SQ-AA/NOPB, U7 AP7384-50SA-7, U8 LMR33630BRNXR, U9 LMR33630BRNXR

Commit message: PVT
Parts:
- removed C41, C44, C49: 100n, Capacitor-Chip:C_CHIP_1005_Hand_NoSilk, symbol passive:C
- removed C46: 1u, Capacitor-Chip:C_CHIP_1005_Hand_NoSilk, symbol passive:C
- removed L4, L5, L8: 100, Inductor-Chip:L_CHIP_1608_Reflow, symbol passive:L_Ferrite
- removed L6: ETQ-P3M2R2KVP, Inductor-Panasonic:PCC-M0530M-LP, symbol passive:L
- removed U8: LMR33630BRNXR, IC-QFN:VQFN12-HR_002, symbol power-ti:LMR33630xRNX
- added U7: TPSM53604RDAR, IC-QFN:B3QFN, symbol power-ti:TPSM53604RDA
- C41: renamed from C38; value 4.7u -> 10u; PartName (none) -> GRM21BC8YA106KE11L
- C42: renamed from C40; value 4.7u -> 10u; PartName (none) -> GRM21BC8YA106KE11L
- C43: renamed from C37; value 4.7u -> 10u; PartName (none) -> GRM21BC8YA106KE11L
- C45: renamed from C39; value 4.7u -> 10u; PartName (none) -> GRM21BC8YA106KE11L
- C47, C58, C59, C62, C67, C68: PartName C1005X5R1V105K050BE -> TMK105BJ105MV-F
- C48: renamed from C43; value 1u(35V) -> 100n; footprint Capacitor-Chip:C_CHIP_1608_Reflow -> Capacitor-Chip:C_CHIP_1005_Hand_NoSilk; PartName GMK107BJ105KAHT -> GRM155R71H104ME14D
- C50: renamed from C48; PartName C1005X5R1V105K050BE -> TMK105BJ105MV-F
- C51: value 22u -> 47u; PartName GRM21BR61E226ME44L -> JMK212BJ476MG-T
- C52: renamed from C54; value 22u -> 47u; PartName GRM21BR61E226ME44L -> JMK212BJ476MG-T
- C54: renamed from C52; PartName ECA-0JM221 -> 6.3ZLH220MEFC5X11
- C56: renamed from C55; PartName ECA-0JM221 -> 6.3ZLH220MEFC5X11
- C57: PartName ECA-0JM221 -> 6.3ZLH220MEFC5X11
- C60, C61, C65, C66: value 10u -> 22u; footprint Capacitor-Chip:C_CHIP_1608_Reflow -> Capacitor-Chip:C_CHIP_2012_Reflow; PartName EMK107BBJ106MA-T -> GRM21BR61E226ME44L
- R32: renamed from R33; value 120k -> 10k; PartName RK73H1ETTP1203F -> RK73H1ETTP1002F
- R33: renamed from R34; value 30k -> 2.49k; PartName RK73H1ETTP3002F -> RK73H1ETTP2491F; Supplier P板 -> (none)
- R36: renamed from R41; value 470k -> 430k; PartName RK73H1ETTP4703F -> RK73H1ETTP4303F
- R37: renamed from R42; value 180k -> 160k; PartName RK73H1ETTP1803F -> RK73H1ETTP1603F
- R40: renamed from R37; value 470k -> 430k; PartName RK73H1ETTP4703F -> RK73H1ETTP4303F
- R41: renamed from R38; value 120k -> 110k; PartName RK73H1ETTP1203F -> RK73H1ETTP1103F
- R42: renamed from R39; value 560k -> 430k; PartName RK73H1ETTP5603F -> RK73H1ETTP4303F
- R43: renamed from R40; value 100k -> 75k; PartName RK73H1ETTP1003F -> RK73H1ETTP7502F
- U9: renamed from U7; Supplier Mouser -> (none)
- renumbered C42 to C44, C45 to C46, C50 to C49, C56 to C55, L7 to L4, L9 to L5, L10 to L6, R35 to R34, R36 to R35, R43 to R38, R44 to R39, U9 to U8
Connections:
- net 3V3_VIN is gone; now on net VSYS: C41.1, C42.1, C44.1, C46.1, U8.10 (VIN), U8.2 (VIN)
- net 5V_VIN is gone; now on net VSYS: C43.1, C45.1
- net PMIC_VIN is gone; now on net +5V: C58.1, C59.1, C60.1, C61.1, C62.1, D7.2 (A), U10.1 (VINLDO12), U10.10 (AVDD), U10.13 (VIN2), U10.19 (VINLDO1), U10.24 (VINLDO2), U10.6 (VIN1)
- net +5V: now also U7.7 (VOUT), U7.8 (VOUT)
- net GND: now also U7.10 (NC), U7.11 (NC), U7.12 (AGND), U7.15 (PGND), U7.3 (NC)
- net P5V_EN: now also U7.2 (EN)
- net VSYS: now also U7.1 (VIN), U7.14 (VIN)
- net at R32.2, R33.1: now also U7.9 (FB)
- no-connect marks 1 -> 2
Other:
- note added: "VOUT(+1V8)=1.84V\nVOUT(+1V2)=1.19V\nVOUT(+2V5)=2.45V\nVOUT(+3V3A)=3.37V"
- note added: "VOUT(+5V)=5.02V"
- note added: "VSYS to 5V/4A Buck Regulator"
- note removed: "VOUT(+1V8)=1.81V\nVOUT(+1V2)=1.19V\nVOUT(+2V5)=2.46V\nVOUT(+3V3A)=3.30V"
- note removed: "VOUT(+5V)=5.00V"
- note removed: "VSYS to 5V/3A Buck Regulator"
- moved on the sheet: C41, C42, C43, C44, C45, C46, C47, C49, C51, C52, C53, C54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

Commit message: SBUにTVSダイオードを追加
Parts:
- D7: symbol diode:D_PN -> diode:D_Schottkey
Connections:
- no-connect marks 2 -> 4
Changed lines of the file:
@@
 Connection ~ 3600 6500
 $Comp
-L diode:D_PN D?
+L diode:D_Schottkey D?
 U 1 1 5F3C97DD
 P 4800 6500
@@
 Wire Wire Line
 	9100 4800 10300 4800
+NoConn ~ 2600 4500
+NoConn ~ 3400 2000
 $EndSCHEMATC
