File: Processor-Camera.sch (KiCad schematic (older format))
At the start: 18 parts, among them J11 1-84952-5, J12 1-84952-5, U14 TS3A24159DGSR, U15 PESD5V0X1BQ,115, U16 PESD5V0X1BQ,115, U17 PESD5V0X1BQ,115, U18 PESD5V0X1BQ,115, U19 PESD5V0X1BQ,115, U20 PESD5V0X1BQ,115, U21 PESD5V0X1BQ,115, U22 PESD5V0X1BQ,115

Commit message: PVT
Parts:
- J10: renamed from J11; value 1-84952-5 -> 1-84953-5; PartName 1-84952-5 -> 1-84953-5
- J11: renamed from J12; value 1-84952-5 -> 1-84953-5; PartName 1-84952-5 -> 1-84953-5
- renumbered C76 to C72, C77 to C73, R59 to R52, R60 to R53, R61 to R54, R62 to R55, R63 to R56, U14 to U12, U15 to U13, U16 to U14, U17 to U15, U18 to U16, U19 to U17, U20 to U18, U21 to U19, U22 to U20

Commit message: SBUにTVSダイオードを追加
Parts:
- U13, U14, U15, U16, U17, U18, U19, U20: value PESD5V0X1BQ,115 -> PESD5V0X1BQ,115
Changed lines of the file:
@@
 AR Path="/5E724900/5E72F29A/5E79BD0B" Ref="#PWR?"  Part="1"
 AR Path="/5E644AAD/5E79BD0B" Ref="#PWR?"  Part="1"
-AR Path="/5E9E174E/5EC20A75/5E79BD0B" Ref="#PWR0178"  Part="1"
-F 0 "#PWR0178" H 10300 2550 50  0001 C CNN
+AR Path="/5E9E174E/5EC20A75/5E79BD0B" Ref="#PWR0177"  Part="1"
+F 0 "#PWR0177" H 10300 2550 50  0001 C CNN
 F 1 "GND" H 10300 2650 50  0000 C CNN
 F 2 "" H 10300 2800 50  0001 C CNN
@@
 AR Path="/5E724900/5E72F29A/5E79E0FF" Ref="#PWR?"  Part="1"
 AR Path="/5E644AAD/5E79E0FF" Ref="#PWR?"  Part="1"
-AR Path="/5E9E174E/5EC20A75/5E79E0FF" Ref="#PWR0179"  Part="1"
-F 0 "#PWR0179" H 10300 5650 50  0001 C CNN
+AR Path="/5E9E174E/5EC20A75/5E79E0FF" Ref="#PWR0178"  Part="1"
+F 0 "#PWR0178" H 10300 5650 50  0001 C CNN
 F 1 "GND" H 10300 5750 50  0000 C CNN
 F 2 "" H 10300 5900 50  0001 C CNN
@@
 AR Path="/5E724900/5E72F29A/5F0180E1" Ref="#PWR?"  Part="1"
 AR Path="/5E644AAD/5F0180E1" Ref="#PWR?"  Part="1"
-AR Path="/5E9E174E/5EC20A75/5F0180E1" Ref="#PWR0173"  Part="1"
-F 0 "#PWR0173" H 1400 5950 50  0001 C CNN
+AR Path="/5E9E174E/5EC20A75/5F0180E1" Ref="#PWR0172"  Part="1"
+F 0 "#PWR0172" H 1400 5950 50  0001 C CNN
 F 1 "GND" H 1400 6050 50  0000 C CNN
 F 2 "" H 1400 6200 50  0001 C CNN
@@
 AR Path="/5E724900/5E72F29A/5E7A3346" Ref="#PWR?"  Part="1"
 AR Path="/5E644AAD/5E7A3346" Ref="#PWR?"  Part="1"
-AR Path="/5E9E174E/5EC20A75/5E7A3346" Ref="#PWR0176"  Part="1"
-F 0 "#PWR0176" H 9000 2650 50  0001 C CNN
+AR Path="/5E9E174E/5EC20A75/5E7A3346" Ref="#PWR0175"  Part="1"
+F 0 "#PWR0175" H 9000 2650 50  0001 C CNN
 F 1 "+3V3" V 8900 2900 50  0000 C CNN
 F 2 "" H 9000 2800 50  0001 C CNN
@@
 AR Path="/5E9E174E/5EC20A75/5F09EC75" Ref="U15"  Part="1"
 F 0 "U15" H 7000 2950 50  0000 C CNN
-F 1 "PESD5V0X1BQ,115	" H 7000 2450 50  0000 C CNN
+F 1 "PESD5V0X1BQ,115" H 7000 2450 50  0000 C CNN
 F 2 "IC-SOT:SOT663" H 7000 2700 50  0001 C CNN
 F 3 "" H 7000 2700 50  0001 C CNN
@@
 AR Path="/5E9E174E/5EC20A75/5F0A8D07" Ref="U17"  Part="1"
 F 0 "U17" H 7700 2950 50  0000 C CNN
-F 1 "PESD5V0X1BQ,115	" H 7700 2450 50  0000 C CNN
+F 1 "PESD5V0X1BQ,115" H 7700 2450 50  0000 C CNN
 F 2 "IC-SOT:SOT663" H 7700 2700 50  0001 C CNN
 F 3 "" H 7700 2700 50  0001 C CNN
@@
 AR Path="/5E9E174E/5EC20A75/5F0A8F0A" Ref="U19"  Part="1"
 F 0 "U19" H 8400 2950 50  0000 C CNN
-F 1 "PESD5V0X1BQ,115	" H 8400 2450 50  0000 C CNN
+F 1 "PESD5V0X1BQ,115" H 8400 2450 50  0000 C CNN
 F 2 "IC-SOT:SOT663" H 8400 2700 50  0001 C CNN
 F 3 "" H 8400 2700 50  0001 C CNN
@@
 AR Path="/5E9E174E/5EC20A75/5F0C2521" Ref="U16"  Part="1"
 F 0 "U16" H 7000 6050 50  0000 C CNN
-F 1 "PESD5V0X1BQ,115	" H 7000 5550 50  0000 C CNN
+F 1 "PESD5V0X1BQ,115" H 7000 5550 50  0000 C CNN
 F 2 "IC-SOT:SOT663" H 7000 5800 50  0001 C CNN
 F 3 "" H 7000 5800 50  0001 C CNN
@@
 AR Path="/5E9E174E/5EC20A75/5F0C2527" Ref="U18"  Part="1"
 F 0 "U18" H 7700 6050 50  0000 C CNN
-F 1 "PESD5V0X1BQ,115	" H 7700 5550 50  0000 C CNN
+F 1 "PESD5V0X1BQ,115" H 7700 5550 50  0000 C CNN
 F 2 "IC-SOT:SOT663" H 7700 5800 50  0001 C CNN
 F 3 "" H 7700 5800 50  0001 C CNN
@@
 AR Path="/5E9E174E/5EC20A75/5F0C252D" Ref="U20"  Part="1"
 F 0 "U20" H 8400 6050 50  0000 C CNN
-F 1 "PESD5V0X1BQ,115	" H 8400 5550 50  0000 C CNN
+F 1 "PESD5V0X1BQ,115" H 8400 5550 50  0000 C CNN
 F 2 "IC-SOT:SOT663" H 8400 5800 50  0001 C CNN
 F 3 "" H 8400 5800 50  0001 C CNN
@@
 AR Path="/5E724900/5E72F29A/5F0CCAEF" Ref="#PWR?"  Part="1"
 AR Path="/5E644AAD/5F0CCAEF" Ref="#PWR?"  Part="1"
-AR Path="/5E9E174E/5EC20A75/5F0CCAEF" Ref="#PWR0174"  Part="1"
-F 0 "#PWR0174" H 7700 2850 50  0001 C CNN
+AR Path="/5E9E174E/5EC20A75/5F0CCAEF" Ref="#PWR0173"  Part="1"
+F 0 "#PWR0173" H 7700 2850 50  0001 C CNN
 F 1 "GND" H 7700 2950 50  0000 C CNN
 F 2 "" H 7700 3100 50  0001 C CNN
@@
 AR Path="/5E724900/5E72F29A/5F0DCF8F" Ref="#PWR?"  Part="1"
 AR Path="/5E644AAD/5F0DCF8F" Ref="#PWR?"  Part="1"
-AR Path="/5E9E174E/5EC20A75/5F0DCF8F" Ref="#PWR0175"  Part="1"
-F 0 "#PWR0175" H 7700 5950 50  0001 C CNN
+AR Path="/5E9E174E/5EC20A75/5F0DCF8F" Ref="#PWR0174"  Part="1"
+F 0 "#PWR0174" H 7700 5950 50  0001 C CNN
 F 1 "GND" H 7700 6050 50  0000 C CNN
 F 2 "" H 7700 6200 50  0001 C CNN
@@
 AR Path="/5E9E174E/5EC20A75/5F25E24C" Ref="U14"  Part="1"
 F 0 "U14" H 6300 6050 50  0000 C CNN
-F 1 "PESD5V0X1BQ,115	" H 6300 5550 50  0000 C CNN
+F 1 "PESD5V0X1BQ,115" H 6300 5550 50  0000 C CNN
 F 2 "IC-SOT:SOT663" H 6300 5800 50  0001 C CNN
 F 3 "" H 6300 5800 50  0001 C CNN
@@
 AR Path="/5E9E174E/5EC20A75/5F25E640" Ref="U13"  Part="1"
 F 0 "U13" H 6300 2950 50  0000 C CNN
-F 1 "PESD5V0X1BQ,115	" H 6300 2450 50  0000 C CNN
+F 1 "PESD5V0X1BQ,115" H 6300 2450 50  0000 C CNN
 F 2 "IC-SOT:SOT663" H 6300 2700 50  0001 C CNN
 F 3 "" H 6300 2700 50  0001 C CNN
@@
 AR Path="/5E724900/5E72F29A/5E7A0B15" Ref="#PWR?"  Part="1"
 AR Path="/5E644AAD/5E7A0B15" Ref="#PWR?"  Part="1"
-AR Path="/5E9E174E/5EC20A75/5E7A0B15" Ref="#PWR0177"  Part="1"
-F 0 "#PWR0177" H 9000 5750 50  0001 C CNN
+AR Path="/5E9E174E/5EC20A75/5E7A0B15" Ref="#PWR0176"  Part="1"
+F 0 "#PWR0176" H 9000 5750 50  0001 C CNN
 F 1 "+3V3" V 8900 6000 50  0000 C CNN
 F 2 "" H 9000 5900 50  0001 C CNN
@@
 AR Path="/5E724900/5E72F29A/5EE506CA" Ref="#PWR?"  Part="1"
 AR Path="/5E644AAD/5EE506CA" Ref="#PWR?"  Part="1"
-AR Path="/5E9E174E/5EC20A75/5EE506CA" Ref="#PWR0180"  Part="1"
-F 0 "#PWR0180" H 10900 550 50  0001 C CNN
+AR Path="/5E9E174E/5EC20A75/5EE506CA" Ref="#PWR0179"  Part="1"
+F 0 "#PWR0179" H 10900 550 50  0001 C CNN
 F 1 "GND" H 10900 650 50  0000 C CNN
 F 2 "" H 10900 800 50  0001 C CNN
@@
 AR Path="/5E724900/5E72F29A/5EE607D8" Ref="#PWR?"  Part="1"
 AR Path="/5E644AAD/5EE607D8" Ref="#PWR?"  Part="1"
-AR Path="/5E9E174E/5EC20A75/5EE607D8" Ref="#PWR0181"  Part="1"
-F 0 "#PWR0181" H 10900 3650 50  0001 C CNN
+AR Path="/5E9E174E/5EC20A75/5EE607D8" Ref="#PWR0180"  Part="1"
+F 0 "#PWR0180" H 10900 3650 50  0001 C CNN
 F 1 "GND" H 10900 3750 50  0000 C CNN
 F 2 "" H 10900 3900 50  0001 C CNN
@@
 AR Path="/5E724900/5E72F29A/5F036259" Ref="#PWR?"  Part="1"
 AR Path="/5E644AAD/5F036259" Ref="#PWR?"  Part="1"
-AR Path="/5E9E174E/5EC20A75/5F036259" Ref="#PWR0172"  Part="1"
-F 0 "#PWR0172" H 1400 5250 50  0001 C CNN
+AR Path="/5E9E174E/5EC20A75/5F036259" Ref="#PWR0171"  Part="1"
+F 0 "#PWR0171" H 1400 5250 50  0001 C CNN
 F 1 "GND" H 1400 5350 50  0000 C CNN
 F 2 "" H 1400 5500 50  0001 C CNN
@@
 $EndComp
 $Comp
-L supply-value:+3V3 #PWR0171
+L supply-value:+3V3 #PWR0170
 U 1 1 5F03651F
 P 1400 5100
-F 0 "#PWR0171" H 1400 4950 50  0001 C CNN
+F 0 "#PWR0170" H 1400 4950 50  0001 C CNN
 F 1 "+3V3" H 1400 5240 50  0000 C CNN
 F 2 "" H 1400 5100 50  0001 C CNN
