File: Processor-M2.sch (KiCad schematic (older format))
At the start: 10 parts, among them J13 2199119-4, Q10 BSS138W, Q8 BSS138W, Q9 BSS138W

Commit message: PVT
Parts:
- renumbered C78 to C74, C79 to C75, H16 to J12, R64 to R57, R65 to R58, R66 to R59
Connections:
- net PET0+: now also C75.1; no longer C74.1
- net PET0-: now also C74.1; no longer C75.1
Other:
- note added: "TX, RX pairs are polarity reversed."
- note removed: "RX pair is polarity reversed."
- moved on the sheet: C74, C75
Changed lines of the file:
@@
 encoding utf-8
 Sheet 9 24
-Title "Phoenix DVT"
-Date "2020-05-18"
+Title "Phoenix PVT"
+Date "2020-07-19"
 Rev "1"
 Comp ""
@@
 USB_D+
 $Comp
-L supply-alias:GND #PWR0195
+L supply-alias:GND #PWR0183
 U 1 1 5E663E7F
 P 6700 5600
-F 0 "#PWR0195" H 6700 5350 50  0001 C CNN
+F 0 "#PWR0183" H 6700 5350 50  0001 C CNN
 F 1 "GND" H 6700 5450 50  0000 C CNN
 F 2 "" H 6700 5600 50  0001 C CNN
@@
 $EndComp
 $Comp
-L supply-alias:GND #PWR0197
+L supply-alias:GND #PWR0185
 U 1 1 5E664A8A
 P 7400 5600
-F 0 "#PWR0197" H 7400 5350 50  0001 C CNN
+F 0 "#PWR0185" H 7400 5350 50  0001 C CNN
 F 1 "GND" H 7400 5450 50  0000 C CNN
 F 2 "" H 7400 5600 50  0001 C CNN
@@
 $EndComp
 $Comp
-L supply-alias:GND #PWR0196
+L supply-alias:GND #PWR0184
 U 1 1 5E665457
 P 7050 5600
-F 0 "#PWR0196" H 7050 5350 50  0001 C CNN
+F 0 "#PWR0184" H 7050 5350 50  0001 C CNN
 F 1 "GND" H 7050 5450 50  0000 C CNN
 F 2 "" H 7050 5600 50  0001 C CNN
@@
 L passive:C C?
 U 1 1 5E75DBB0
-P 4500 3400
+P 4500 3500
 AR Path="/5E7D4299/5E75DBB0" Ref="C?"  Part="1"
 AR Path="/5E6353A4/5E75DBB0" Ref="C?"  Part="1"
-AR Path="/5E9E174E/5E7A14E6/5E75DBB0" Ref="C78"  Part="1"
-F 0 "C78" V 4450 3300 50  0000 R CNN
-F 1 "100n" V 4450 3500 50  0000 L CNN
-F 2 "Capacitor-Chip:C_CHIP_1005_Hand_NoSilk" H 4600 3300 50  0001 C CNN
-F 3 "" H 4525 3500 50  0001 C CNN
-F 4 "GRM155R71H104ME14D" H 4500 3400 50  0001 C CNN "PartName"
-	1    4500 3400
+AR Path="/5E9E174E/5E7A14E6/5E75DBB0" Ref="C74"  Part="1"
+F 0 "C74" V 4450 3400 50  0000 R CNN
+F 1 "100n" V 4450 3600 50  0000 L CNN
+F 2 "Capacitor-Chip:C_CHIP_1005_Hand_NoSilk" H 4600 3400 50  0001 C CNN
+F 3 "" H 4525 3600 50  0001 C CNN
+F 4 "GRM155R71H104ME14D" H 4500 3500 50  0001 C CNN "PartName"
+	1    4500 3500
 	0    1    1    0
 $EndComp
@@
 L passive:C C?
 U 1 1 5E75FF24
-P 5000 3500
+P 5000 3400
 AR Path="/5E7D4299/5E75FF24" Ref="C?"  Part="1"
 AR Path="/5E6353A4/5E75FF24" Ref="C?"  Part="1"
-AR Path="/5E9E174E/5E7A14E6/5E75FF24" Ref="C79"  Part="1"
-F 0 "C79" V 4950 3400 50  0000 R CNN
-F 1 "100n" V 4950 3600 50  0000 L CNN
-F 2 "Capacitor-Chip:C_CHIP_1005_Hand_NoSilk" H 5100 3400 50  0001 C CNN
-F 3 "" H 5025 3600 50  0001 C CNN
-F 4 "GRM155R71H104ME14D" H 5000 3500 50  0001 C CNN "PartName"
-	1    5000 3500
+AR Path="/5E9E174E/5E7A14E6/5E75FF24" Ref="C75"  Part="1"
+F 0 "C75" V 4950 3300 50  0000 R CNN
+F 1 "100n" V 4950 3500 50  0000 L CNN
+F 2 "Capacitor-Chip:C_CHIP_1005_Hand_NoSilk" H 5100 3300 50  0001 C CNN
+F 3 "" H 5025 3500 50  0001 C CNN
+F 4 "GRM155R71H104ME14D" H 5000 3400 50  0001 C CNN "PartName"
+	1    5000 3400
 	0    1    1    0
 $EndComp
 Wire Wire Line
-	4000 3500 4900 3500
+	4000 3400 4900 3400
 Text Notes 4400 5800 0    50   ~ 0
 2199119-4 + 9774015243R\n  1.5 mm Bottom Spacing\n  Total 3.2 mm Height\n\n2199230-4 + 9774025243R\n  2.5 mm Bottom Spacing\n  Total 4.2mm Height
@@
 Text HLabel 9500 4700 2    50   Input ~ 0
 W_DISABLE1
+Text HLabel 4000 3500 0    50   Input ~ 0
+PCIE_TX0+
 Text HLabel 4000 3400 0    50   Input ~ 0
-PCIE_TX0+
-Text HLabel 4000 3500 0    50   Input ~ 0
 PCIE_TX0-
 Text HLabel 4000 3800 0    50   Output ~ 0
@@
 ~PERST0
 $Comp
-L supply-value:+3V3 #PWR0198
+L supply-value:+3V3 #PWR0186
 U 1 1 5E7B5A87
 P 7500 1700
-F 0 "#PWR0198" H 7500 1550 50  0001 C CNN
+F 0 "#PWR0186" H 7500 1550 50  0001 C CNN
 F 1 "+3V3" H 7500 1840 50  0000 C CNN
 F 2 "" H 7500 1700 50  0001 C CNN
@@
 	4000 3800 6800 3800
 Wire Wire Line
-	5100 3500 6800 3500
-Wire Wire Line
-	4600 3400 6800 3400
-Wire Wire Line
-	4400 3400 4000 3400
+	5100 3400 6800 3400
+Wire Wire Line
+	4600 3500 6800 3500
+Wire Wire Line
+	4400 3500 4000 3500
 Wire Wire Line
 	4000 4400 6800 4400
@@
 	8700 4700 9500 4700
 $Comp
-L supply-alias:GND #PWR0201
+L supply-alias:GND #PWR0189
 U 1 1 5E875EDE
 P 8500 5200
-F 0 "#PWR0201" H 8500 4950 50  0001 C CNN
+F 0 "#PWR0189" H 8500 4950 50  0001 C CNN
 F 1 "GND" H 8500 5050 50  0000 C CNN
 F 2 "" H 8500 5200 50  0001 C CNN
@@
 $EndComp
 $Comp
-L supply-alias:GND #PWR0204
+L supply-alias:GND #PWR0192
 U 1 1 5E87605A
 P 9000 5200
-F 0 "#PWR0204" H 9000 4950 50  0001 C CNN
+F 0 "#PWR0192" H 9000 4950 50  0001 C CNN
 F 1 "GND" H 9000 5050 50  0000 C CNN
 F 2 "" H 9000 5200 50  0001 C CNN
@@
 Connection ~ 9000 4300
 $Comp
-L passive:R R65
+L passive:R R58
 U 1 1 5E879B4F
 P 8500 4100
-F 0 "R65" H 8550 4150 50  0000 L CNN
+F 0 "R58" H 8550 4150 50  0000 L CNN
 F 1 "10k" H 8550 4050 50  0000 L CNN
 F 2 "Resistor-Chip:R_CHIP_1005_Hand_NoSilk" V 8550 4000 50  0001 C CNN
@@
 $EndComp
 $Comp
-L passive:R R66
+L passive:R R59
 U 1 1 5E879C80
 P 9000 4100
-F 0 "R66" H 9050 4150 50  0000 L CNN
+F 0 "R59" H 9050 4150 50  0000 L CNN
 F 1 "10k" H 9050 4050 50  0000 L CNN
 F 2 "Resistor-Chip:R_CHIP_1005_Hand_NoSilk" V 9050 4000 50  0001 C CNN
@@
 $EndComp
 $Comp
-L supply-value:+3V3 #PWR0200
+L supply-value:+3V3 #PWR0188
 U 1 1 5E879E88
 P 8500 4000
-F 0 "#PWR0200" H 8500 3850 50  0001 C CNN
+F 0 "#PWR0188" H 8500 3850 50  0001 C CNN
 F 1 "+3V3" H 8500 4140 50  0000 C CNN
 F 2 "" H 8500 4000 50  0001 C CNN
@@
 $EndComp
 $Comp
-L supply-value:+3V3 #PWR0203
+L supply-value:+3V3 #PWR0191
 U 1 1 5E87B302
 P 9000 4000
-F 0 "#PWR0203" H 9000 3850 50  0001 C CNN
+F 0 "#PWR0191" H 9000 3850 50  0001 C CNN
 F 1 "+3V3" H 9000 4140 50  0000 C CNN
 F 2 "" H 9000 4000 50  0001 C CNN
@@
 $EndComp
 $Comp
-L print:MountPad H16
+L print:MountPad J12
 U 1 1 5EAD3D13
 P 6000 5400
-F 0 "H16" V 5735 5400 50  0000 C CNN
+F 0 "J12" V 5735 5400 50  0000 C CNN
 F 1 "9774015243R" V 5826 5400 50  0000 C CNN
 F 2 "Phoenix:9774015243R" H 6000 5400 50  0001 C CNN
@@
 $EndComp
 $Comp
-L supply-alias:GND #PWR0194
+L supply-alias:GND #PWR0182
 U 1 1 5EAD42A6
 P 6000 5600
-F 0 "#PWR0194" H 6000 5350 50  0001 C CNN
+F 0 "#PWR0182" H 6000 5350 50  0001 C CNN
 F 1 "GND" H 6000 5450 50  0000 C CNN
 F 2 "" H 6000 5600 50  0001 C CNN
@@
 $EndComp
 $Comp
-L supply-value:+1V8 #PWR0202
+L supply-value:+1V8 #PWR0190
 U 1 1 5FB473C3
 P 9000 3100
-F 0 "#PWR0202" H 9000 2950 50  0001 C CNN
+F 0 "#PWR0190" H 9000 2950 50  0001 C CNN
 F 1 "+1V8" H 9000 3240 50  0000 C CNN
 F 2 "" H 9000 3100 50  0001 C CNN
@@
 SUSCLK
 $Comp
-L passive:R R64
+L passive:R R57
 U 1 1 5FB4A452
 P 8500 3100
-F 0 "R64" H 8550 3150 50  0000 L CNN
+F 0 "R57" H 8550 3150 50  0000 L CNN
 F 1 "10k" H 8550 3050 50  0000 L CNN
 F 2 "Resistor-Chip:R_CHIP_1005_Hand_NoSilk" V 8550 3000 50  0001 C CNN
@@
 $EndComp
 $Comp
-L supply-value:+3V3 #PWR0199
+L supply-value:+3V3 #PWR0187
 U 1 1 5FB4AA02
 P 8500 3000
-F 0 "#PWR0199" H 8500 2850 50  0001 C CNN
+F 0 "#PWR0187" H 8500 2850 50  0001 C CNN
 F 1 "+3V3" H 8500 3140 50  0000 C CNN
 F 2 "" H 8500 3000 50  0001 C CNN
@@
 	6700 2000 6700 3300
 Text Notes 3500 3200 0    50   ~ 0
-RX pair is polarity reversed.
+TX, RX pairs are polarity reversed.
 $EndSCHEMATC
