File: Phoenix.sch (KiCad schematic (older format))
At the start: 27 parts

Commit message: FPGA_INTをFPGA_MODEに変更
Changed lines of the file:
@@
 F90 "FPGA_SPI_MOSI" I L 9000 2700 50
 F91 "FPGA_SPI_MISO" O L 9000 2800 50
-F92 "FPGA_INT" O L 9000 2200 50
+F92 "FPGA_MODE" I L 9000 2200 50
 F93 "MOTOR1_LED" O L 9000 6200 50
 F94 "MOTOR2_LED" O L 9000 6300 50
@@
 	2000 1300 4000 1300
 Text Label 6200 2200 0    50   ~ 0
-GPIO12_FPGA_INT
+GPIO12_FPGA_MODE
 Wire Wire Line
 	2000 1500 2200 1500
